File: electronic/kc_car_boards/kc_car_boards.sch (KiCad schematic (older format))
At the start: 3 parts, among them J6 SPI3, J7 SPI2, J8 SPI1

Commit message: scheme update
Parts:
- renumbered J6 to J1, J7 to J2, J8 to J3
Changed lines of the file:
@@
 	2750 2800 3500 2800
 $Comp
-L Connector:Conn_01x04_Male J6
+L Connector:Conn_01x04_Male J1
 U 1 1 5DB1E135
 P 2150 4550
-F 0 "J6" H 2122 4432 50  0000 R CNN
+F 0 "J1" H 2122 4432 50  0000 R CNN
 F 1 "SPI3" H 2122 4523 50  0000 R CNN
 F 2 "Connector_PinHeader_2.54mm:PinHeader_1x04_P2.54mm_Vertical" H 2150 4550 50  0001 C CNN
@@
 $EndComp
 $Comp
-L Connector:Conn_01x04_Male J7
+L Connector:Conn_01x04_Male J2
 U 1 1 5DB227B2
 P 2150 5100
-F 0 "J7" H 2122 4982 50  0000 R CNN
+F 0 "J2" H 2122 4982 50  0000 R CNN
 F 1 "SPI2" H 2122 5073 50  0000 R CNN
 F 2 "Connector_PinHeader_2.54mm:PinHeader_1x04_P2.54mm_Vertical" H 2150 5100 50  0001 C CNN
@@
 $EndComp
 $Comp
-L Connector:Conn_01x04_Male J8
+L Connector:Conn_01x04_Male J3
 U 1 1 5DB22E53
 P 2150 5600
-F 0 "J8" H 2122 5482 50  0000 R CNN
+F 0 "J3" H 2122 5482 50  0000 R CNN
 F 1 "SPI1" H 2122 5573 50  0000 R CNN
 F 2 "Connector_PinHeader_2.54mm:PinHeader_1x04_P2.54mm_Vertical" H 2150 5600 50  0001 C CNN
