File: electronic/kc_car_boards/microcontroller.sch (KiCad schematic (older format))
At the start: 5 parts, among them J3 FTDI, U4 Atmega328, Y1 16MHz

Commit message: scheme update
Parts:
- C5, C6: footprint (none) -> Capacitor_SMD:C_0805_2012Metric_Pad1.15x1.40mm_HandSolder
- renumbered J3 to J6
Changed lines of the file:
@@
 $EndComp
 $Comp
-L power:GNDD #PWR0102
+L power:GNDD #PWR09
 U 1 1 5DAE86F6
 P 5300 4750
-F 0 "#PWR0102" H 5300 4500 50  0001 C CNN
+F 0 "#PWR09" H 5300 4500 50  0001 C CNN
 F 1 "GNDD" H 5304 4595 50  0000 C CNN
 F 2 "" H 5300 4750 50  0001 C CNN
@@
 $EndComp
 $Comp
-L power:+5V #PWR0103
+L power:+5V #PWR03
 U 1 1 5DAE8DDB
 P 5250 1900
-F 0 "#PWR0103" H 5250 1750 50  0001 C CNN
+F 0 "#PWR03" H 5250 1750 50  0001 C CNN
 F 1 "+5V" H 5265 2073 50  0000 C CNN
 F 2 "" H 5250 1900 50  0001 C CNN
@@
 F 0 "C6" H 5592 2096 50  0000 L CNN
 F 1 "0.1uF" H 5592 2005 50  0000 L CNN
-F 2 "" H 5500 2050 50  0001 C CNN
+F 2 "Capacitor_SMD:C_0805_2012Metric_Pad1.15x1.40mm_HandSolder" H 5500 2050 50  0001 C CNN
 F 3 "~" H 5500 2050 50  0001 C CNN
 	1    5500 2050
@@
 $EndComp
 $Comp
-L power:GNDD #PWR0104
+L power:GNDD #PWR05
 U 1 1 5DAEABEB
 P 5700 2200
-F 0 "#PWR0104" H 5700 1950 50  0001 C CNN
+F 0 "#PWR05" H 5700 1950 50  0001 C CNN
 F 1 "GNDD" H 5704 2045 50  0000 C CNN
 F 2 "" H 5700 2200 50  0001 C CNN
@@
 	5250 2050 5250 2300
 $Comp
-L power:GNDD #PWR0105
+L power:GNDD #PWR04
 U 1 1 5DAEBD30
 P 4800 2200
-F 0 "#PWR0105" H 4800 1950 50  0001 C CNN
+F 0 "#PWR04" H 4800 1950 50  0001 C CNN
 F 1 "GNDD" H 4804 2045 50  0000 C CNN
 F 2 "" H 4800 2200 50  0001 C CNN
@@
 $EndComp
 $Comp
-L power:+5V #PWR0106
+L power:+5V #PWR02
 U 1 1 5DAEC1D3
 P 4800 1700
-F 0 "#PWR0106" H 4800 1550 50  0001 C CNN
+F 0 "#PWR02" H 4800 1550 50  0001 C CNN
 F 1 "+5V" H 4815 1873 50  0000 C CNN
 F 2 "" H 4800 1700 50  0001 C CNN
@@
 F 0 "C5" H 4892 1996 50  0000 L CNN
 F 1 "0.1uF" H 4892 1905 50  0000 L CNN
-F 2 "" H 4800 1950 50  0001 C CNN
+F 2 "Capacitor_SMD:C_0805_2012Metric_Pad1.15x1.40mm_HandSolder" H 4800 1950 50  0001 C CNN
 F 3 "~" H 4800 1950 50  0001 C CNN
 	1    4800 1950
@@
 	4050 3250 4600 3250
 $Comp
-L power:GNDD #PWR0107
+L power:GNDD #PWR07
 U 1 1 5DAEEFAA
 P 4150 3600
-F 0 "#PWR0107" H 4150 3350 50  0001 C CNN
+F 0 "#PWR07" H 4150 3350 50  0001 C CNN
 F 1 "GNDD" H 4154 3445 50  0000 C CNN
 F 2 "" H 4150 3600 50  0001 C CNN
@@
 	4150 3600 4150 3450
 $Comp
-L Connector:Conn_01x04_Male J3
+L Connector:Conn_01x04_Male J6
 U 1 1 5DAF01C9
 P 7500 3500
-F 0 "J3" H 7472 3474 50  0000 R CNN
+F 0 "J6" H 7472 3474 50  0000 R CNN
 F 1 "FTDI" H 7472 3383 50  0000 R CNN
 F 2 "" H 7500 3500 50  0001 C CNN
@@
 $EndComp
 $Comp
-L power:GNDD #PWR0108
+L power:GNDD #PWR08
 U 1 1 5DAF0B1F
 P 7200 3800
-F 0 "#PWR0108" H 7200 3550 50  0001 C CNN
+F 0 "#PWR08" H 7200 3550 50  0001 C CNN
 F 1 "GNDD" H 7204 3645 50  0000 C CNN
 F 2 "" H 7200 3800 50  0001 C CNN
@@
 $EndComp
 $Comp
-L power:+5V #PWR0109
+L power:+5V #PWR06
 U 1 1 5DAF1243
 P 7200 3300
-F 0 "#PWR0109" H 7200 3150 50  0001 C CNN
+F 0 "#PWR06" H 7200 3150 50  0001 C CNN
 F 1 "+5V" H 7215 3473 50  0000 C CNN
 F 2 "" H 7200 3300 50  0001 C CNN
