File: electronic/kc_car_boards/mosfets.sch (KiCad schematic (older format))
At the start: 8 parts, among them J4 Load1, J5 Load2, Q1 IRF540N, Q2 IRF540N

Commit message: scheme update
Parts:
- R1, R2, R3, R4: footprint (none) -> Resistor_SMD:R_0805_2012Metric_Pad1.15x1.40mm_HandSolder
- renumbered J4 to J7, J5 to J8
Changed lines of the file:
@@
 $EndComp
 $Comp
-L power:GNDD #PWR0110
+L power:GNDD #PWR012
 U 1 1 5DB06EDA
 P 3650 2500
-F 0 "#PWR0110" H 3650 2250 50  0001 C CNN
+F 0 "#PWR012" H 3650 2250 50  0001 C CNN
 F 1 "GNDD" H 3654 2345 50  0000 C CNN
 F 2 "" H 3650 2500 50  0001 C CNN
@@
 F 0 "R1" V 2843 1800 50  0000 C CNN
 F 1 "100" V 2934 1800 50  0000 C CNN
-F 2 "" V 2980 1800 50  0001 C CNN
+F 2 "Resistor_SMD:R_0805_2012Metric_Pad1.15x1.40mm_HandSolder" V 2980 1800 50  0001 C CNN
 F 3 "~" H 3050 1800 50  0001 C CNN
 	1    3050 1800
@@
 F 0 "R3" H 3370 2196 50  0000 L CNN
 F 1 "10K" H 3370 2105 50  0000 L CNN
-F 2 "" V 3230 2150 50  0001 C CNN
+F 2 "Resistor_SMD:R_0805_2012Metric_Pad1.15x1.40mm_HandSolder" V 3230 2150 50  0001 C CNN
 F 3 "~" H 3300 2150 50  0001 C CNN
 	1    3300 2150
@@
 $EndComp
 $Comp
-L power:GNDD #PWR0111
+L power:GNDD #PWR013
 U 1 1 5DB0CEA5
 P 5450 2500
-F 0 "#PWR0111" H 5450 2250 50  0001 C CNN
+F 0 "#PWR013" H 5450 2250 50  0001 C CNN
 F 1 "GNDD" H 5454 2345 50  0000 C CNN
 F 2 "" H 5450 2500 50  0001 C CNN
@@
 F 0 "R2" V 4643 1800 50  0000 C CNN
 F 1 "100" V 4734 1800 50  0000 C CNN
-F 2 "" V 4780 1800 50  0001 C CNN
+F 2 "Resistor_SMD:R_0805_2012Metric_Pad1.15x1.40mm_HandSolder" V 4780 1800 50  0001 C CNN
 F 3 "~" H 4850 1800 50  0001 C CNN
 	1    4850 1800
@@
 F 0 "R4" H 5170 2196 50  0000 L CNN
 F 1 "10K" H 5170 2105 50  0000 L CNN
-F 2 "" V 5030 2150 50  0001 C CNN
+F 2 "Resistor_SMD:R_0805_2012Metric_Pad1.15x1.40mm_HandSolder" V 5030 2150 50  0001 C CNN
 F 3 "~" H 5100 2150 50  0001 C CNN
 	1    5100 2150
@@
 	5450 1350 5450 1600
 $Comp
-L Connector:Conn_01x02_Male J4
+L Connector:Conn_01x02_Male J7
 U 1 1 5DB16F7B
 P 3650 1150
-F 0 "J4" V 3712 1194 50  0000 L CNN
+F 0 "J7" V 3712 1194 50  0000 L CNN
 F 1 "Load1" V 3803 1194 50  0000 L CNN
 F 2 "Connector_PinHeader_2.54mm:PinHeader_1x02_P2.54mm_Vertical" H 3650 1150 50  0001 C CNN
@@
 $EndComp
 $Comp
-L Connector:Conn_01x02_Male J5
+L Connector:Conn_01x02_Male J8
 U 1 1 5DB17BDB
 P 5450 1150
-F 0 "J5" V 5512 1194 50  0000 L CNN
+F 0 "J8" V 5512 1194 50  0000 L CNN
 F 1 "Load2" V 5603 1194 50  0000 L CNN
 F 2 "Connector_PinHeader_2.54mm:PinHeader_1x02_P2.54mm_Vertical" H 5450 1150 50  0001 C CNN
@@
 $EndComp
 $Comp
-L power:VCC #PWR0112
+L power:VCC #PWR010
 U 1 1 5DB18207
 P 3200 1000
-F 0 "#PWR0112" H 3200 850 50  0001 C CNN
+F 0 "#PWR010" H 3200 850 50  0001 C CNN
 F 1 "VCC" H 3217 1173 50  0000 C CNN
 F 2 "" H 3200 1000 50  0001 C CNN
@@
 $EndComp
 $Comp
-L power:VCC #PWR0113
+L power:VCC #PWR011
 U 1 1 5DB188BD
 P 5200 1000
-F 0 "#PWR0113" H 5200 850 50  0001 C CNN
+F 0 "#PWR011" H 5200 850 50  0001 C CNN
 F 1 "VCC" H 5217 1173 50  0000 C CNN
 F 2 "" H 5200 1000 50  0001 C CNN
