File: electronic/kc_car_boards/motors_controller.sch (KiCad schematic (older format))
At the start: 12 parts, among them J1 Motor1, J2 Motor2, U3 L298HN

Commit message: scheme update
Parts:
- renumbered J1 to J4, J2 to J5
Changed lines of the file:
@@
 $EndComp
 $Comp
-L Connector:Screw_Terminal_01x02 J1
+L Connector:Screw_Terminal_01x02 J4
 U 1 1 5DAC4332
 P 5050 1800
-F 0 "J1" H 5130 1792 50  0000 L CNN
+F 0 "J4" H 5130 1792 50  0000 L CNN
 F 1 "Motor1" H 5130 1701 50  0000 L CNN
 F 2 "TerminalBlock:TerminalBlock_bornier-2_P5.08mm" H 5050 1800 50  0001 C CNN
@@
 $EndComp
 $Comp
-L Connector:Screw_Terminal_01x02 J2
+L Connector:Screw_Terminal_01x02 J5
 U 1 1 5DAC4DCC
 P 5050 2100
-F 0 "J2" H 5130 2092 50  0000 L CNN
+F 0 "J5" H 5130 2092 50  0000 L CNN
 F 1 "Motor2" H 5130 2001 50  0000 L CNN
 F 2 "TerminalBlock:TerminalBlock_bornier-2_P5.08mm" H 5050 2100 50  0001 C CNN
