File: electronic/kc_car_boards/police_sound.sch (KiCad schematic (older format))
At the start: 14 parts

Commit message: scheme update
Parts:
- C10, C9: renamed from C?; footprint (none) -> Capacitor_THT:CP_Radial_D12.5mm_P7.50mm
- C11: renamed from C?; footprint (none) -> Capacitor_THT:C_Disc_D14.5mm_W5.0mm_P10.00mm
- C7: renamed from C?; footprint (none) -> Capacitor_SMD:C_0805_2012Metric_Pad1.15x1.40mm_HandSolder
- C8: renamed from C?; footprint (none) -> Capacitor_THT:CP_Radial_D8.0mm_P5.00mm
- R5, R6, R7, R8, R9: renamed from R?; footprint (none) -> Resistor_SMD:R_0805_2012Metric_Pad1.15x1.40mm_HandSolder
- U5, U6: renamed from U?; footprint (none) -> libs:SOIC-8_W3.9mm
- gave numbers to parts that had none: 2
Connections:
- net GND: now also C10.1; no longer C10.2
- net at R7.2, U6.5 (CONT): now also C10.2; no longer C10.1
Changed lines of the file:
@@
 $EndDescr
 $Comp
-L abby:NE555 U?
+L abby:NE555 U5
 U 1 1 5DAB8147
 P 3350 1950
-F 0 "U?" H 3100 2350 50  0000 C CNN
+F 0 "U5" H 3100 2350 50  0000 C CNN
 F 1 "NE555" H 3550 2350 50  0000 C CNN
-F 2 "" H 3350 1950 50  0001 C CNN
+F 2 "libs:SOIC-8_W3.9mm" H 3350 1950 50  0001 C CNN
 F 3 "http://www.ti.com/lit/ds/symlink/ne555.pdf" H 3350 1950 50  0001 C CNN
 	1    3350 1950
@@
 $EndComp
 $Comp
-L abby:NE555 U?
+L abby:NE555 U6
 U 1 1 5DAB8AEA
 P 3350 4100
-F 0 "U?" H 3100 4450 50  0000 C CNN
+F 0 "U6" H 3100 4450 50  0000 C CNN
 F 1 "NE555" H 3550 4450 50  0000 C CNN
-F 2 "" H 3350 4100 50  0001 C CNN
+F 2 "libs:SOIC-8_W3.9mm" H 3350 4100 50  0001 C CNN
 F 3 "http://www.ti.com/lit/ds/symlink/ne555.pdf" H 3350 4100 50  0001 C CNN
 	1    3350 4100
@@
 Connection ~ 3350 1450
 $Comp
-L power:VCC #PWR?
+L power:VCC #PWR014
 U 1 1 5DABB894
 P 3350 1150
-F 0 "#PWR?" H 3350 1000 50  0001 C CNN
+F 0 "#PWR014" H 3350 1000 50  0001 C CNN
 F 1 "VCC" H 3367 1323 50  0000 C CNN
 F 2 "" H 3350 1150 50  0001 C CNN
@@
 $EndComp
 $Comp
-L power:GND #PWR?
+L power:GND #PWR016
 U 1 1 5DABBEB8
 P 3350 2800
-F 0 "#PWR?" H 3350 2550 50  0001 C CNN
+F 0 "#PWR016" H 3350 2550 50  0001 C CNN
 F 1 "GND" H 3355 2627 50  0000 C CNN
 F 2 "" H 3350 2800 50  0001 C CNN
@@
 $EndComp
 $Comp
-L Device:C_Small C?
+L Device:C_Small C7
 U 1 1 5DABC770
 P 2500 2150
-F 0 "C?" H 2592 2196 50  0000 L CNN
+F 0 "C7" H 2592 2196 50  0000 L CNN
 F 1 "0.1uF" H 2592 2105 50  0000 L CNN
-F 2 "" H 2500 2150 50  0001 C CNN
+F 2 "Capacitor_SMD:C_0805_2012Metric_Pad1.15x1.40mm_HandSolder" H 2500 2150 50  0001 C CNN
 F 3 "~" H 2500 2150 50  0001 C CNN
 	1    2500 2150
@@
 	3350 2400 3350 2350
 $Comp
-L Device:R R?
+L Device:R R5
 U 1 1 5DABD153
 P 4500 1700
-F 0 "R?" H 4570 1746 50  0000 L CNN
+F 0 "R5" H 4570 1746 50  0000 L CNN
 F 1 "1K" H 4570 1655 50  0000 L CNN
-F 2 "" V 4430 1700 50  0001 C CNN
+F 2 "Resistor_SMD:R_0805_2012Metric_Pad1.15x1.40mm_HandSolder" V 4430 1700 50  0001 C CNN
 F 3 "~" H 4500 1700 50  0001 C CNN
 	1    4500 1700
@@
 $EndComp
 $Comp
-L Device:R R?
+L Device:R R6
 U 1 1 5DABDC3C
 P 4500 2200
-F 0 "R?" H 4570 2246 50  0000 L CNN
+F 0 "R6" H 4570 2246 50  0000 L CNN
 F 1 "10K" H 4570 2155 50  0000 L CNN
-F 2 "" V 4430 2200 50  0001 C CNN
+F 2 "Resistor_SMD:R_0805_2012Metric_Pad1.15x1.40mm_HandSolder" V 4430 2200 50  0001 C CNN
 F 3 "~" H 4500 2200 50  0001 C CNN
 	1    4500 2200
@@
 $EndComp
 $Comp
-L Device:CP_Small C?
+L Device:CP_Small C8
 U 1 1 5DABE6B5
 P 4500 2650
-F 0 "C?" H 4588 2696 50  0000 L CNN
+F 0 "C8" H 4588 2696 50  0000 L CNN
 F 1 "68uF" H 4588 2605 50  0000 L CNN
-F 2 "" H 4500 2650 50  0001 C CNN
+F 2 "Capacitor_THT:CP_Radial_D8.0mm_P5.00mm" H 4500 2650 50  0001 C CNN
 F 3 "~" H 4500 2650 50  0001 C CNN
 	1    4500 2650
@@
 $EndComp
 $Comp
-L Device:CP_Small C?
+L Device:CP_Small C11
 U 1 1 5DABF29C
 P 4250 4800
-F 0 "C?" H 4338 4846 50  0000 L CNN
+F 0 "C11" H 4338 4846 50  0000 L CNN
 F 1 "0,047uF" H 4338 4755 50  0000 L CNN
-F 2 "" H 4250 4800 50  0001 C CNN
+F 2 "Capacitor_THT:C_Disc_D14.5mm_W5.0mm_P10.00mm" H 4250 4800 50  0001 C CNN
 F 3 "~" H 4250 4800 50  0001 C CNN
 	1    4250 4800
@@
 $EndComp
 $Comp
-L Device:CP_Small C?
+L Device:CP_Small C10
 U 1 1 5DABF8F7
 P 2350 4600
-F 0 "C?" H 2438 4646 50  0000 L CNN
+F 0 "C10" H 2438 4646 50  0000 L CNN
 F 1 "100uF" H 2438 4555 50  0000 L CNN
-F 2 "" H 2350 4600 50  0001 C CNN
+F 2 "Capacitor_THT:CP_Radial_D12.5mm_P7.50mm" H 2350 4600 50  0001 C CNN
 F 3 "~" H 2350 4600 50  0001 C CNN
 	1    2350 4600
-	1    0    0    -1
-$EndComp
-$Comp
-L Device:R R?
+	1    0    0    1
+$EndComp
+$Comp
+L Device:R R7
 U 1 1 5DAC03C4
 P 2350 3550
-F 0 "R?" H 2420 3596 50  0000 L CNN
+F 0 "R7" H 2420 3596 50  0000 L CNN
 F 1 "1K" H 2420 3505 50  0000 L CNN
-F 2 "" V 2280 3550 50  0001 C CNN
+F 2 "Resistor_SMD:R_0805_2012Metric_Pad1.15x1.40mm_HandSolder" V 2280 3550 50  0001 C CNN
 F 3 "~" H 2350 3550 50  0001 C CNN
 	1    2350 3550
@@
 $EndComp
 $Comp
-L Device:R R?
+L Device:R R8
 U 1 1 5DAC099D
 P 4250 3800
-F 0 "R?" H 4320 3846 50  0000 L CNN
+F 0 "R8" H 4320 3846 50  0000 L CNN
 F 1 "1K" H 4320 3755 50  0000 L CNN
-F 2 "" V 4180 3800 50  0001 C CNN
+F 2 "Resistor_SMD:R_0805_2012Metric_Pad1.15x1.40mm_HandSolder" V 4180 3800 50  0001 C CNN
 F 3 "~" H 4250 3800 50  0001 C CNN
 	1    4250 3800
@@
 $EndComp
 $Comp
-L Device:R R?
+L Device:R R9
 U 1 1 5DAC130C
 P 4250 4350
-F 0 "R?" H 4320 4396 50  0000 L CNN
+F 0 "R9" H 4320 4396 50  0000 L CNN
 F 1 "10K" H 4320 4305 50  0000 L CNN
-F 2 "" V 4180 4350 50  0001 C CNN
+F 2 "Resistor_SMD:R_0805_2012Metric_Pad1.15x1.40mm_HandSolder" V 4180 4350 50  0001 C CNN
 F 3 "~" H 4250 4350 50  0001 C CNN
 	1    4250 4350
@@
 	3350 1200 3350 1150
 $Comp
-L power:VCC #PWR?
+L power:VCC #PWR018
 U 1 1 5DAC7470
 P 3350 3350
-F 0 "#PWR?" H 3350 3200 50  0001 C CNN
+F 0 "#PWR018" H 3350 3200 50  0001 C CNN
 F 1 "VCC" H 3367 3523 50  0000 C CNN
 F 2 "" H 3350 3350 50  0001 C CNN
@@
 $EndComp
 $Comp
-L power:GND #PWR?
+L power:GND #PWR021
 U 1 1 5DAC7C40
 P 3350 5200
-F 0 "#PWR?" H 3350 4950 50  0001 C CNN
+F 0 "#PWR021" H 3350 4950 50  0001 C CNN
 F 1 "GND" H 3355 5027 50  0000 C CNN
 F 2 "" H 3350 5200 50  0001 C CNN
@@
 	3350 3350 3350 3650
 $Comp
-L Connector:Conn_01x02_Male J?
+L Connector:Conn_01x02_Male J10
 U 1 1 5DAC9DBC
 P 4100 3150
-F 0 "J?" V 4162 3194 50  0000 L CNN
+F 0 "J10" V 4162 3194 50  0000 L CNN
 F 1 "Buzzer" V 4253 3194 50  0000 L CNN
 F 2 "Connector_PinHeader_2.54mm:PinHeader_1x02_P2.54mm_Vertical" H 4100 3150 50  0001 C CNN
@@
 	4000 3900 4000 3350
 $Comp
-L power:GND #PWR?
+L power:GND #PWR019
 U 1 1 5DACB729
 P 4100 3550
-F 0 "#PWR?" H 4100 3300 50  0001 C CNN
+F 0 "#PWR019" H 4100 3300 50  0001 C CNN
 F 1 "GND" H 4105 3377 50  0000 C CNN
 F 2 "" H 4100 3550 50  0001 C CNN
@@
 	4100 3550 4100 3350
 $Comp
-L power:VCC #PWR?
+L power:VCC #PWR020
 U 1 1 5DACC7C4
 P 4250 3550
-F 0 "#PWR?" H 4250 3400 50  0001 C CNN
+F 0 "#PWR020" H 4250 3400 50  0001 C CNN
 F 1 "VCC" H 4267 3723 50  0000 C CNN
 F 2 "" H 4250 3550 50  0001 C CNN
@@
 Connection ~ 4050 4600
 $Comp
-L Device:CP_Small C?
+L Device:CP_Small C9
 U 1 1 5DAD9664
 P 6250 2750
-F 0 "C?" H 6338 2796 50  0000 L CNN
+F 0 "C9" H 6338 2796 50  0000 L CNN
 F 1 "100uF" H 6338 2705 50  0000 L CNN
-F 2 "" H 6250 2750 50  0001 C CNN
+F 2 "Capacitor_THT:CP_Radial_D12.5mm_P7.50mm" H 6250 2750 50  0001 C CNN
 F 3 "~" H 6250 2750 50  0001 C CNN
 	1    6250 2750
@@
 $EndComp
 $Comp
-L power:VCC #PWR?
+L power:VCC #PWR015
 U 1 1 5DAD9C8C
 P 6250 2400
-F 0 "#PWR?" H 6250 2250 50  0001 C CNN
+F 0 "#PWR015" H 6250 2250 50  0001 C CNN
 F 1 "VCC" H 6267 2573 50  0000 C CNN
 F 2 "" H 6250 2400 50  0001 C CNN
@@
 $EndComp
 $Comp
-L power:GND #PWR?
+L power:GND #PWR017
 U 1 1 5DADA1F3
 P 6250 3050
-F 0 "#PWR?" H 6250 2800 50  0001 C CNN
+F 0 "#PWR017" H 6250 2800 50  0001 C CNN
 F 1 "GND" H 6255 2877 50  0000 C CNN
 F 2 "" H 6250 3050 50  0001 C CNN
@@
 $EndComp
 $Comp
-L Connector:Conn_01x02_Male J?
+L Connector:Conn_01x02_Male J9
 U 1 1 5DADAE39
 P 7000 2800
-F 0 "J?" H 6972 2682 50  0000 R CNN
+F 0 "J9" H 6972 2682 50  0000 R CNN
 F 1 "Power" H 6972 2773 50  0000 R CNN
 F 2 "Connector_PinHeader_2.54mm:PinHeader_1x02_P2.54mm_Vertical" H 7000 2800 50  0001 C CNN
